Commit message: fix(z1_urdf): lower joint2_PositionMin from 0.0 to -pi/2 to account for offset
With joint_offset=1.57 applied, the physical flat position maps to TRUE=1.57.
The old min=0.0 prevented IK from finding solutions below TRUE=1.57.
New min=-1.57 allows the IK to explore the full reachable range.

File: src/z1_ros2/z1_description/urdf/const.xacro (robot description, xacro)
@@ -109,5 +109,5 @@
     <xacro:property name="joint1_PositionMin" value="${-PI*150/180}"/>
     <xacro:property name="joint1_PositionMax" value="${PI*150/180}"/>
-    <xacro:property name="joint2_PositionMin" value="0.0"/>
+    <xacro:property name="joint2_PositionMin" value="${-PI*90/180}"/>
     <xacro:property name="joint2_PositionMax" value="${PI*170/180}"/>
     <xacro:property name="joint3_PositionMin" value="${-PI*165/180}"/>

Commit message: revert: restore joint2_PositionMin to 0.0

File: src/z1_ros2/z1_description/urdf/const.xacro (robot description, xacro)
@@ -109,5 +109,5 @@
     <xacro:property name="joint1_PositionMin" value="${-PI*150/180}"/>
     <xacro:property name="joint1_PositionMax" value="${PI*150/180}"/>
-    <xacro:property name="joint2_PositionMin" value="${-PI*90/180}"/>
+    <xacro:property name="joint2_PositionMin" value="0.0"/>
     <xacro:property name="joint2_PositionMax" value="${PI*170/180}"/>
     <xacro:property name="joint3_PositionMin" value="${-PI*165/180}"/>
