Commit message: fix: remove duplicate Grey material, add SpotYellow for Spot body/legs
- Removed Grey material definition from spotzi.urdf.xacro (already in z1_macro.xacro)
- Added SpotYellow material (rgba 0.96 0.82 0.15) with references to all
  13 Spot visual links (body + 4x hip/upper_leg/lower_leg)
- Fixes urdfdom 'material not unique' error in Jazzy/Humble

File: src/spotzi_description/urdf/spot_macro.xacro (robot description, xacro)
@@ -14,4 +14,5 @@
                     <mesh filename="package://spotzi_description/meshes/base/visual/body.obj" />
                 </geometry>
+                <material name="SpotYellow"/>
             </visual>
             <collision>
@@ -66,4 +67,5 @@
                         filename="package://spotzi_description/meshes/base/visual/front_left_hip.obj" />
                 </geometry>
+                <material name="SpotYellow"/>
             </visual>
             <inertial>
@@ -100,4 +102,5 @@
                         filename="package://spotzi_description/meshes/base/visual/front_left_upper_leg.obj" />
                 </geometry>
+                <material name="SpotYellow"/>
             </visual>
             <collision>
@@ -140,4 +143,5 @@
                         filename="package://spotzi_description/meshes/base/visual/front_left_lower_leg.obj" />
                 </geometry>
+                <material name="SpotYellow"/>
             </visual>
             <collision>
@@ -186,4 +190,5 @@
                         filename="package://spotzi_description/meshes/base/visual/front_right_hip.obj" />
                 </geometry>
+                <material name="SpotYellow"/>
             </visual>
             <inertial>
@@ -220,4 +225,5 @@
                         filename="package://spotzi_description/meshes/base/visual/front_right_upper_leg.obj" />
                 </geometry>
+                <material name="SpotYellow"/>
             </visual>
             <collision>
@@ -260,4 +266,5 @@
                         filename="package://spotzi_description/meshes/base/visual/front_right_lower_leg.obj" />
                 </geometry>
+                <material name="SpotYellow"/>
             </visual>
             <collision>
@@ -306,4 +313,5 @@
                         filename="package://spotzi_description/meshes/base/visual/rear_left_hip.obj" />
                 </geometry>
+                <material name="SpotYellow"/>
             </visual>
             <inertial>
@@ -340,4 +348,5 @@
                         filename="package://spotzi_description/meshes/base/visual/rear_left_upper_leg.obj" />
                 </geometry>
+                <material name="SpotYellow"/>
             </visual>
             <collision>
@@ -380,4 +389,5 @@
                         filename="package://spotzi_description/meshes/base/visual/rear_left_lower_leg.obj" />
                 </geometry>
+                <material name="SpotYellow"/>
             </visual>
             <collision>
@@ -426,4 +436,5 @@
                         filename="package://spotzi_description/meshes/base/visual/rear_right_hip.obj" />
                 </geometry>
+                <material name="SpotYellow"/>
             </visual>
             <inertial>
@@ -460,4 +471,5 @@
                         filename="package://spotzi_description/meshes/base/visual/rear_right_upper_leg.obj" />
                 </geometry>
+                <material name="SpotYellow"/>
             </visual>
             <collision>
@@ -500,4 +512,5 @@
                         filename="package://spotzi_description/meshes/base/visual/rear_right_lower_leg.obj" />
                 </geometry>
+                <material name="SpotYellow"/>
             </visual>
             <collision>

File: src/spotzi_description/urdf/spotzi.urdf.xacro (robot description, xacro)
@@ -27,6 +27,6 @@
   <!-- Materials                                                         -->
   <!-- ================================================================= -->
-  <material name="Grey">
-    <color rgba="0.3 0.3 0.3 1.0" />
+  <material name="SpotYellow">
+    <color rgba="0.96 0.82 0.15 1.0" />
   </material>
   <!-- ================================================================= -->
